File: design/pcb_design/STM32G041F8P6_dev.kicad_pcb (KiCad board)
At the start: 4 copper layers, 27 parts, among them J1 USB_B_Micro, J2 Conn_02x02_Odd_Even, J3 S2B-PH-K-S, J4 Conn_ST_STDC14, SW1 Reset, U1 MIC5301-3.3YD5, U2 STM32G041F8Px, U3 MCP73831-2-OT, Y1 Crystal

Commit message: updates to pcb
Parts:
- added C11: 0.1uF, Capacitor_SMD:C_0805_2012Metric, F.Cu at (144.3, 56.0)
- added C12: 0.1uF, Capacitor_SMD:C_0805_2012Metric, F.Cu at (144.3, 59.0)
- added CR1: LSM115JE3/TR13, _custom:DO-214BA_MCH, F.Cu at (163.0, 50.0)
- added CR2: LSM115JE3/TR13, _custom:DO-214BA_MCH, F.Cu at (208.0, 90.0)
- added R10: 10K, Resistor_SMD:R_0805_2012Metric, F.Cu at (134.2, 61.7)
- added R5: 470, Resistor_SMD:R_0805_2012Metric, F.Cu at (129.8, 61.7)
- added R6: 10K, Resistor_SMD:R_0805_2012Metric, F.Cu at (134.2, 49.9)
- added R7: 10K, Resistor_SMD:R_0805_2012Metric, F.Cu at (134.2, 52.9)
- added R8: 10K, Resistor_SMD:R_0805_2012Metric, F.Cu at (134.2, 55.8)
- added R9: 10K, Resistor_SMD:R_0805_2012Metric, F.Cu at (134.2, 58.8)
- added SW2: 2-1825910-7, _custom:SW4_1825910-G_TEC, F.Cu at (171.6, 76.2)
- added SW3: 2-1825910-7, _custom:SW4_1825910-G_TEC, F.Cu at (194.2, 76.4)
- added SW4: 2-1825910-7, _custom:SW4_1825910-G_TEC, F.Cu at (218.0, 76.5)
- added U4: ADXL343BCCZ, Package_LGA:LGA-14_3x5mm_P0.8mm_LayoutBorder1x6y, F.Cu at (168.0, 88.4)
- C1: value 12.5pF -> 0.1uF
- C10: value 1uF -> 1uF CER
- C2: value 12.5pF -> 4.7uF; footprint Capacitor_SMD:C_0603_1608Metric -> Capacitor_SMD:C_1206_3216Metric
- C3: value 0.1uF -> 12.5pF
- C4: value 4.7nF 1KV -> 12.5pF; footprint Capacitor_SMD:C_0805_2012Metric -> Capacitor_SMD:C_0603_1608Metric
- C5: value 0.1uF -> 4.7nF 1KV; footprint Capacitor_SMD:C_0603_1608Metric -> Capacitor_SMD:C_0805_2012Metric
- C6: value 1uF CER -> 0.1uF; footprint Capacitor_SMD:C_1206_3216Metric -> Capacitor_SMD:C_0603_1608Metric
- C7: value 0.01uF -> 1uF CER; footprint Capacitor_SMD:C_0805_2012Metric -> Capacitor_SMD:C_1206_3216Metric
- C8: value 1uF CER -> 1uF
- C9: value 4.7uF -> 0.01uF; footprint Capacitor_SMD:C_1206_3216Metric -> Capacitor_SMD:C_0805_2012Metric
- D1: value LSM115JE3 -> Power; footprint Diode_SMD:D_SMC -> LED_SMD:LED_0805_2012Metric
- D2: value LSM115JE3 -> Green Indicator; footprint Diode_SMD:D_SMC -> LED_SMD:LED_0805_2012Metric
- D3: value Power -> Red indicator
- D4: value Power -> SSD1306; footprint LED_SMD:LED_0805_2012Metric -> _custom:SmallOLED
- J2: value Conn_02x02_Odd_Even -> S2B-PH-K-S; footprint Connector_PinHeader_2.54mm:PinHeader_2x02_P2.54mm_Vertical -> Connector_JST:JST_PH_S2B-PH-K_1x02_P2.00mm_Horizontal
- J3: value S2B-PH-K-S -> Conn_02x02_Odd_Even; footprint Connector_JST:JST_PH_S2B-PH-K_1x02_P2.00mm_Horizontal -> Connector_PinHeader_2.54mm:PinHeader_2x02_P2.54mm_Vertical
- R2: value 100 -> 5K
- U1: value MIC5301-3.3YD5 -> MCP73831-2-OT; footprint Package_TO_SOT_SMD:TSOT-23-5 -> Package_TO_SOT_SMD:SOT-23-5
- U2: value STM32G041F8Px -> MIC5301-3.3YD5; footprint Package_SO:TSSOP-20_4.4x6.5mm_P0.65mm -> Package_TO_SOT_SMD:TSOT-23-5
- U3: value MCP73831-2-OT -> STM32G041F8Px; footprint Package_TO_SOT_SMD:SOT-23-5 -> Package_SO:TSSOP-20_4.4x6.5mm_P0.65mm
- moved D3 88.5 mm to (203.0, 68.0)
- moved J3 85.8 mm to (189.5, 88.5)
- moved J2 83.0 mm to (217.0, 86.0), turned to 90 degrees
- moved D2 82.9 mm to (180.0, 67.8)
- moved J1 62.5 mm to (158.3, 58.0), turned to -90 degrees
- moved D1 53.8 mm to (143.0, 83.0)
- moved SW1 46.4 mm to (108.3, 89.7)
- moved C6 42.5 mm to (137.6, 80.2)
- moved C9 39.2 mm to (144.3, 53.0)
- moved Y1 39.1 mm to (113.7, 89.2)
- moved U1 37.2 mm to (138.1, 83.9)
- moved D4 35.7 mm to (178.3, 58.0), turned to -90 degrees
- moved C10 33.7 mm to (139.3, 60.2)
- moved C8 33.7 mm to (139.3, 56.8)
- moved U3 29.7 mm to (130.7, 86.4)
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Connections:
- C1 pad 1: Net-(U2-PC14/PB9) -> +3.3V
- C10 pad 1: Net-(J3-Pin_2) -> GND
- C10 pad 2: GND -> +3.3V
- C2 pad 1: Net-(U2-PC15) -> VBUS
- C3 pad 1: +3.3V -> Net-(U3-PC14/PB9)
- C4 pad 1: Net-(J1-Shield) -> Net-(U3-PC15)
- C5 pad 1: Net-(J4-~{RST}) -> Net-(J1-Shield)
- C6 pad 1: GND -> Net-(J4-~{RST})
- C6 pad 2: Net-(D1-K) -> GND
- C7 pad 1: Net-(U1-BYP) -> GND
- C7 pad 2: GND -> Net-(U2-EN)
- C8 pad 1: GND -> Net-(J2-Pin_2)
- C8 pad 2: +3.3V -> GND
- C9 pad 1: VBUS -> Net-(U2-BYP)
- D2 pad 1: Net-(D1-K) -> Net-(D2-K)
- D2 pad 2: +BATT -> /PA0
- D3 pad 2: VBUS -> /PA1
- D4 pad 1: GND -> SDA
- D4 pad 2: Net-(D4-A) -> SCL
- J2 pad 1: /USART2_TX -> GND
- J2 pad 2: /VCP_TX -> Net-(J2-Pin_2)
- J3 pad 1: GND -> /USART2_TX
- J3 pad 2: Net-(J3-Pin_2) -> /VCP_TX
- R2 pad 1: Net-(U3-PROG) -> Net-(U1-PROG)
- R3 pad 1: Net-(U3-STAT) -> Net-(U1-STAT)
- R3 pad 2: Net-(D3-K) -> Net-(D1-K)
- R4 pad 1: +3.3V -> GND
- R4 pad 2: Net-(D4-A) -> Net-(D2-K)
- U1 pad 1: Net-(D1-K) -> Net-(U1-STAT)
- U1 pad 3: Net-(D1-K) -> Net-(J2-Pin_2)
- U1 pad 4: Net-(U1-BYP) -> VBUS
- U1 pad 5: +3.3V -> Net-(U1-PROG)
- U2 pad 1: unconnected-(U2-PB7/PB8-Pad1) -> Net-(U2-EN)
- U2 pad 2: Net-(U2-PC14/PB9) -> GND
- U2 pad 3: Net-(U2-PC15) -> Net-(U2-EN)
- U2 pad 4: +3.3V -> Net-(U2-BYP)
- U2 pad 5: GND -> +3.3V
- U3 pad 1: Net-(U3-STAT) -> SDA
- U3 pad 2: GND -> Net-(U3-PC14/PB9)
- U3 pad 3: Net-(J3-Pin_2) -> Net-(U3-PC15)
- U3 pad 4: VBUS -> +3.3V
- U3 pad 5: Net-(U3-PROG) -> GND
- Y1 pad 1: Net-(U2-PC14/PB9) -> Net-(U3-PC14/PB9)
- Y1 pad 2: Net-(U2-PC15) -> Net-(U3-PC15)
Other:
- board outline added: 70 x 50 mm

Commit message: pcb updates, initial layout
Parts:
- added H1: MountingHole, MountingHole:MountingHole_3.2mm_M3, F.Cu at (159.5, 49.5)
- added H2: MountingHole, MountingHole:MountingHole_3.2mm_M3, F.Cu at (222.5, 49.5)
- added H3: MountingHole, MountingHole:MountingHole_3.2mm_M3, F.Cu at (159.5, 92.5)
- added H4: MountingHole, MountingHole:MountingHole_3.2mm_M3, F.Cu at (222.5, 92.5)
- J2, J3: moved to B.Cu
- SW2: value 2-1825910-7 -> Up
- SW3: value 2-1825910-7 -> Enter
- SW4: value 2-1825910-7 -> Down
- moved R3 91.8 mm to (215.3, 89.2)
- moved R8 89.3 mm to (221.7, 73.8)
- moved C2 88.4 mm to (220.2, 85.7)
- moved R2 87.4 mm to (212.8, 80.3)
- moved C8 85.7 mm to (221.2, 81.8)
- moved Y1 75.5 mm to (189.1, 83.9)
- moved U1 72.9 mm to (211.1, 84.2)
- moved R5 72.7 mm to (202.0, 70.7)
- moved D1 72.6 mm to (215.0, 92.0)
- moved SW1 72.0 mm to (179.8, 81.1)
- moved R7 68.2 mm to (199.1, 74.1)
- moved U3 64.8 mm to (195.4, 88.3)
- moved R4 55.1 mm to (184.3, 67.3)
- moved C1 54.6 mm to (190.1, 87.7), turned to -90 degrees
- moved C4 51.2 mm to (187.4, 89.4)
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Routing:
- net Net-(U3-PC15): track 0.00 -> 5.89 mm
- net Net-(U3-PC14/PB9): track 0.00 -> 3.48 mm
- net GND: track 0.00 -> 2.62 mm
- net +3.3V: track 0.00 -> 2.62 mm

Commit message: pcb updates
Parts:
- moved R1 68.2 mm to (223.7, 76.8), turned to 180 degrees
- moved J1 68.1 mm to (223.3, 82.5), turned to 90 degrees
- moved C5 63.7 mm to (223.7, 74.7), turned to 180 degrees
- moved CR1 51.9 mm to (216.5, 80.9), turned to 0 degrees
- moved J3 49.8 mm to (182.4, 89.6)
- moved C7 47.1 mm to (201.2, 88.2), turned to 90 degrees
- moved U2 45.9 mm to (204.5, 86.7)
- moved C10 44.3 mm to (206.7, 83.6), turned to 180 degrees
- moved C9 40.7 mm to (207.8, 86.7), turned to 90 degrees
- moved U4 38.7 mm to (197.2, 91.3)
- moved D2 38.5 mm to (216.7, 56.0), turned to 180 degrees
- moved R4 38.3 mm to (220.9, 56.0), turned to 180 degrees
- moved C12 30.8 mm to (193.5, 90.9)
- moved R5 21.7 mm to (220.9, 60.0), turned to 180 degrees
- moved D3 15.9 mm to (216.7, 60.0), turned to 180 degrees
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Connections:
- C8 pad 1: Net-(J2-Pin_2) -> +BATT
- J2 pad 2: Net-(J2-Pin_2) -> +BATT
- SW2 pad 3: +3V3 -> +3.3V
- SW2 pad 4: +3V3 -> +3.3V
- SW3 pad 3: +3V3 -> +3.3V
- SW3 pad 4: +3V3 -> +3.3V
- SW4 pad 3: +3V3 -> +3.3V
- SW4 pad 4: +3V3 -> +3.3V
- U1 pad 3: Net-(J2-Pin_2) -> +BATT
Routing:
- net /PA1: track 0.00 -> 64.4 mm, vias 0 -> 2
- net SDA: track 0.00 -> 54.2 mm, vias 0 -> 2
- net GND: track 2.62 -> 54.1 mm, vias 0 -> 22
- net SCL: track 0.00 -> 49.2 mm, vias 0 -> 3
- net /PA0: track 0.00 -> 45.6 mm, vias 0 -> 4
- net /PA6: track 0.00 -> 41.8 mm, vias 0 -> 2
- net /PA4: track 0.00 -> 36.8 mm
- net Net-(J4-~{RST}): track 0.00 -> 35.8 mm, vias 0 -> 2
- net /PA5: track 0.00 -> 31.7 mm
- net Net-(U2-EN): track 0.00 -> 29.9 mm
- net /SWDIO: track 0.00 -> 27.5 mm, vias 0 -> 2
- net +3.3V: track 2.62 -> 29.4 mm, vias 0 -> 7
- net /SWCLK: track 0.00 -> 26.6 mm, vias 0 -> 2
- net VBUS: track 0.00 -> 18.1 mm
- net Net-(J1-Shield): track 0.00 -> 17.1 mm
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- added copper zone on In2.Cu, net +3.3V
- added copper zone on B.Cu, net GND
- added copper zone on F.Cu, net GND
- added copper zone on In1.Cu, net GND
- added copper zone on F.Cu, net VBUS

Commit message: Update STM32G041F8P6_dev.kicad_pcb
Routing:
- net Net-(J4-~{RST}): track 35.8 -> 35.1 mm

Commit message: PCB Design Updates
Parts:
- added R11: 10K, Resistor_SMD:R_0805_2012Metric, F.Cu at (217.8, 77.5)
- moved C3 1.32 mm to (179.2, 78.3)
- moved C4 1.30 mm to (179.2, 80.8)
- moved Y1 1.26 mm to (181.9, 79.6)
- moved C1 0.08 mm to (182.9, 83.5)
Routing:
- net GND: track 54.1 -> 62.7 mm, vias 22 -> 26
- net VBUS: track 18.1 -> 21.1 mm
- net +3.3V: track 29.4 -> 31.0 mm
- net Net-(U3-PC15): track 6.28 -> 5.12 mm

Commit message: Final changes before manufacture.
Parts:
- C11, C12: footprint Capacitor_SMD:C_0805_2012Metric -> Capacitor_SMD:C_0603_1608Metric
Routing:
- net +3.3V: track 31.0 -> 31.7 mm
Other:
- board text added: "+"
- board text added: "-"
- board text added: "UR"
- board text added: "UT"
- board text added: "VR"
- board text added: "VT"
