File: design/pcb_design/STM32G041F8P6_dev.kicad_sch (KiCad schematic)
At the start: 33 parts, among them J1 USB_B_Micro, J2 Conn_02x02_Odd_Even, J3 S2B-PH-K-S, J4 Conn_ST_STDC14, SW1 Reset, SW2 Reset, U1 MIC5301-3.3YD5, U2 STM32G041F8Px, U3 MCP73831-2-OT, U4 ADXL343BCCZ, Y1 Crystal

Commit message: updates!
Parts:
- removed D5: Power, LED_SMD:LED_0805_2012Metric, symbol Device:LED
- removed R4: 470, Resistor_SMD:R_0805_2012Metric, symbol Device:R_US
- added R10, R8, R9: 10K, symbol Device:R_Small_US
- added R6, R7: 10K, Resistor_SMD:R_0805_2012Metric, symbol Device:R_US
- added SW3: Enter, symbol Switch:SW_Push
- added SW4: Down, symbol Switch:SW_Push
- added SW5: Up, symbol Switch:SW_Push
- R2: value 100 -> 5K
Connections:
- net PA10_12 is gone; now on net AI2: U2.17 (PA12/PA10)
- net PA9_11 is gone; now on net AI1: U2.16 (PA11/PA9)
- net +3.3V: now also R6.2, R7.2
- net GND: now also R10.1, R8.1, R9.1
- net PA5: now also R10.2, SW4.2
- net PA6: now also R9.2, SW3.2
- net PA7: now also R8.2, SW5.2
- net SCL: now also R7.1
- net SDA: now also R6.1
- new net +3V3: SW3.1, SW4.1, SW5.1
Other:
- note added: "Charge Rate 200mA"
- note added: "I2C Pullups"
- note added: "INT Push-Pull"
- note added: "MCU Bypass Ceramic"
- moved on the sheet: C1, C10, C11, C12, C2, C3, C4, C6, C7, C8, C9, D1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

Commit message: updates to pcb
Parts:
- removed D1, D2: LSM115JE3, Diode_SMD:D_SMC, symbol Device:D_Small
- removed SW2: Reset, Button_Switch_SMD:SW_SPST_B3U-1000P, symbol Switch:SW_Push
- removed SW3: Enter, symbol Switch:SW_Push
- removed SW4: Down, symbol Switch:SW_Push
- removed SW5: Up, symbol Switch:SW_Push
- added CR1, CR2: LSM115JE3/TR13, _custom:DO-214BA_MCH, symbol _custom:LSM115JE3_TR13
- added D2: Green Indicator, LED_SMD:LED_0805_2012Metric, symbol Device:LED
- added D3: Red indicator, LED_SMD:LED_0805_2012Metric, symbol Device:LED
- added R4: 470, Resistor_SMD:R_0805_2012Metric, symbol Device:R_US
- added SW2, SW3, SW4: 2-1825910-7, _custom:SW4_1825910-G_TEC, symbol _custom:2-1825910-7
- R5: value 10K -> 470
- R6: renamed from R8; footprint (none) -> Resistor_SMD:R_0805_2012Metric
- R7: renamed from R9; footprint (none) -> Resistor_SMD:R_0805_2012Metric
- R8: renamed from R10; footprint (none) -> Resistor_SMD:R_0805_2012Metric
- renumbered C3 to C1, C8 to C10, C12 to C11, C11 to C12, C9 to C2, C1 to C3, C2 to C4, C4 to C5, C5 to C6, C6 to C7, C10 to C8, C7 to C9, D3 to D1, J3 to J2, J2 to J3, R7 to R10, R6 to R9, U3 to U1, U1 to U2, U2 to U3
Connections:
- net +3V3: now also SW2.3, SW2.4, SW3.3, SW3.4, SW4.3, SW4.4
- net +BATT: now also CR2.2
- net AI1: now also U3.14 (PA7); no longer U3.16 (PA11/PA9)
- net AI2: now also U3.16 (PA11/PA9); no longer U3.17 (PA12/PA10)
- net GND: now also R4.1
- net PA0: now also D2.2 (A)
- net PA1: now also D3.2 (A)
- net PA4: now also R8.2, SW4.1, SW4.2; no longer R5.2
- net PA5: now also R7.2, SW3.1, SW3.2; no longer R8.2
- net PA6: now also R6.2, SW2.1, SW2.2; no longer R7.2
- net SCL: now also U3.20 (PB3/PB4/PB5/PB6)
- net SDA: now also U3.1 (PB7/PB8)
- net VBUS: now also CR1.2
- net at C7.2, U2.1 (VIN), U2.3 (EN): now also CR1.1, CR2.1
- removed net PA7: R6.2, U3.14 (PA7)
- new net: D2.1 (K), R4.2
- new net: D3.1 (K), R5.2
- new net PA10_12: U3.17 (PA12/PA10)
- no-connect marks 11 -> 10
Other:
- note removed: "Check footprints"
- moved on the sheet: C3, C4, R6, R7, R8, Y1

Commit message: pcb updates, initial layout
Parts:
- added H1, H2, H3, H4: MountingHole, MountingHole:MountingHole_3.2mm_M3, symbol Mechanical:MountingHole
- SW2: value 2-1825910-7 -> Up
- SW3: value 2-1825910-7 -> Enter
- SW4: value 2-1825910-7 -> Down
Other:
- moved on the sheet: R6, R7, R8, SW2, SW3, SW4

Commit message: pcb updates
Connections:
- net +3V3 is gone; now on net +3.3V: SW2.3, SW2.4, SW3.3, SW3.4, SW4.3, SW4.4
- net +BATT: now also C8.1, J2.2 (Pin_2), U1.3 (V_{BAT})
Changed lines of the file:
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@@
+	)
+	(symbol
+		(lib_id "power:+BATT")
+		(at 71.12 176.53 0)
+		(unit 1)
+		(exclude_from_sim no)
+		(in_bom yes)
+		(on_board yes)
+		(dnp no)
+		(property "Reference" "#PWR027"
+			(at 71.12 180.34 0)
+			(effects
+				(font
+					(size 1.27 1.27)
+				)
+				(hide yes)
+			)
+		)
+		(property "Value" "+BATT"
+			(at 71.12 172.72 0)
+			(effects
+				(font
+					(size 1.27 1.27)
+				)
+			)
+		)
+		(property "Footprint" ""
+			(at 71.12 176.53 0)
+			(effects
+				(font
+					(size 1.27 1.27)
+				)
+				(hide yes)
+			)
+		)
+		(property "Datasheet" ""
+			(at 71.12 176.53 0)
+			(effects
+				(font
+					(size 1.27 1.27)
+				)
+				(hide yes)
+			)
+		)
+		(property "Description" "Power symbol creates a global label with name \"+BATT\""
+			(at 71.12 176.53 0)
+			(effects
+				(font
+					(size 1.27 1.27)
+				)
+				(hide yes)
+			)
+		)
+		(pin "1"
+		)
+		(instances
+			(project "STM32G041F8P6_dev"
+				(path "/ee3d00c1-aeff-4118-bd3d-d070c1c83a88"
+					(reference "#PWR027")
+					(unit 1)
+				)
+			)
+		)
 	)
 	(symbol
@@
 		(on_board yes)
 		(dnp no)
-		(fields_autoplaced yes)
 		(property "Reference" "#FLG01"
 			(at 74.93 174.625 0)
@@
 		)
 		(property "Value" "PWR_FLAG"
-			(at 74.93 171.45 0)
+			(at 74.93 170.434 0)
 			(effects
 				(font
@@
 				(path "/ee3d00c1-aeff-4118-bd3d-d070c1c83a88"
 					(reference "C4")
+					(unit 1)
+				)
+			)
+		)
+	)
+	(symbol
+		(lib_id "power:+3.3V")
+		(at 106.68 162.56 0)
+		(unit 1)
+		(exclude_from_sim no)
+		(in_bom yes)
+		(on_board yes)
+		(dnp no)
+		(fields_autoplaced yes)
+		(property "Reference" "#PWR015"
+			(at 106.68 166.37 0)
+			(effects
+				(font
+					(size 1.27 1.27)
+				)
+				(hide yes)
+			)
+		)
+		(property "Value" "+3.3V"
+			(at 106.68 157.48 0)
+			(effects
+				(font
+					(size 1.27 1.27)
+				)
+			)
+		)
+		(property "Footprint" ""
+			(at 106.68 162.56 0)
+			(effects
+				(font
+					(size 1.27 1.27)
+				)
+				(hide yes)
+			)
+		)
+		(property "Datasheet" ""
+			(at 106.68 162.56 0)
+			(effects
+				(font
+					(size 1.27 1.27)
+				)
+				(hide yes)
+			)
+		)
+		(property "Description" "Power symbol creates a global label with name \"+3.3V\""
+			(at 106.68 162.56 0)
+			(effects
+				(font
+					(size 1.27 1.27)
+				)
+				(hide yes)
+			)
+		)
+		(pin "1"
+		)
+		(instances
+			(project "STM32G041F8P6_dev"
+				(path "/ee3d00c1-aeff-4118-bd3d-d070c1c83a88"
+					(reference "#PWR015")
 					(unit 1)
 				)
@@
 					(unit 1)
 				)
-			)
-		)
-	)
-	(symbol
-		(lib_id "power:+3V3")
-		(at 106.68 162.56 0)
-		(unit 1)
-		(exclude_from_sim no)
-		(in_bom yes)
-		(on_board yes)
-		(dnp no)
-		(fields_autoplaced yes)
-		(property "Reference" "#PWR015"
-			(at 106.68 166.37 0)
-			(effects
-				(font
-					(size 1.27 1.27)
-				)
-				(hide yes)
-			)
-		)
-		(property "Value" "+3V3"
-			(at 106.68 157.48 0)
-			(effects
-				(font
-					(size 1.27 1.27)
-				)
-			)
-		)
-		(property "Footprint" ""
-			(at 106.68 162.56 0)
-			(effects
-				(font
-					(size 1.27 1.27)
-				)
-				(hide yes)
-			)
-		)
-		(property "Datasheet" ""
-			(at 106.68 162.56 0)
-			(effects
-				(font
-					(size 1.27 1.27)
-				)
-				(hide yes)
-			)
-		)
-		(property "Description" "Power symbol creates a global label with name \"+3V3\""
-			(at 106.68 162.56 0)
-			(effects
-				(font
-					(size 1.27 1.27)
-				)
-				(hide yes)
-			)
-		)
-		(pin "1"
-		)
-		(instances
-			(project "STM32G041F8P6_dev"
-				(path "/ee3d00c1-aeff-4118-bd3d-d070c1c83a88"
-					(reference "#PWR015")
-					(unit 1)
-				)

Commit message: PCB Design Updates
Parts:
- added R11: 10K, Resistor_SMD:R_0805_2012Metric, symbol Device:R_Small_US
Connections:
- net GND: now also R11.1
- net VBUS: now also R11.2
Changed lines of the file:
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@@
 	)
 	(junction
+		(at 43.18 125.73)
+		(diameter 0)
+		(color 0 0 0 0)
+	)
+	(junction
 		(at 26.67 189.23)
 		(diameter 0)
@@
 	)
 	(symbol
+		(lib_id "power:GND")
+		(at 43.18 130.81 0)
+		(unit 1)
+		(exclude_from_sim no)
+		(in_bom yes)
+		(on_board yes)
+		(dnp no)
+		(fields_autoplaced yes)
+		(property "Reference" "#PWR028"
+			(at 43.18 137.16 0)
+			(effects
+				(font
+					(size 1.27 1.27)
+				)
+				(hide yes)
+			)
+		)
+		(property "Value" "GND"
+			(at 43.18 135.89 0)
+			(effects
+				(font
+					(size 1.27 1.27)
+				)
+			)
+		)
+		(property "Footprint" ""
+			(at 43.18 130.81 0)
+			(effects
+				(font
+					(size 1.27 1.27)
+				)
+				(hide yes)
+			)
+		)
+		(property "Datasheet" ""
+			(at 43.18 130.81 0)
+			(effects
+				(font
+					(size 1.27 1.27)
+				)
+				(hide yes)
+			)
+		)
+		(property "Description" "Power symbol creates a global label with name \"GND\" , ground"
+			(at 43.18 130.81 0)
+			(effects
+				(font
+					(size 1.27 1.27)
+				)
+				(hide yes)
+			)
+		)
+		(pin "1"
+		)
+		(instances
+			(project "STM32G041F8P6_dev"
+				(path "/ee3d00c1-aeff-4118-bd3d-d070c1c83a88"
+					(reference "#PWR028")
+					(unit 1)
+				)
+			)
+		)
+	)
+	(symbol
 		(lib_id "Connector:Conn_ST_STDC14")
 		(at 194.31 74.93 270)
@@
 					(unit 1)
 				)
+			)
+		)
+	)
+	(symbol
+		(lib_id "Device:R_Small_US")
+		(at 43.18 128.27 180)
+		(unit 1)
+		(exclude_from_sim no)
+		(in_bom yes)
+		(on_board yes)
+		(dnp no)
+		(fields_autoplaced yes)
+		(property "Reference" "R11"
+			(at 45.72 126.9999 0)
+			(effects
+				(font
+					(size 1.27 1.27)
+				)
+				(justify right)
+			)
+		)
+		(property "Value" "10K"
+			(at 45.72 129.5399 0)
+			(effects
+				(font
+					(size 1.27 1.27)
+				)
+				(justify right)
+			)
+		)
+		(property "Footprint" "Resistor_SMD:R_0805_2012Metric"
+			(at 43.18 128.27 0)
+			(effects
+				(font
+					(size 1.27 1.27)
+				)
+				(hide yes)
+			)
+		)
+		(property "Datasheet" "~"
+			(at 43.18 128.27 0)
+			(effects
+				(font
+					(size 1.27 1.27)
+				)
+				(hide yes)
+			)
+		)
+		(property "Description" "Resistor, small US symbol"
+			(at 43.18 128.27 0)
+			(effects
+				(font
+					(size 1.27 1.27)
+				)
+				(hide yes)
+			)
+		)
+		(pin "2"
+		)
+		(pin "1"
+		)
+		(instances
+			(project "STM32G041F8P6_dev"
+				(path "/ee3d00c1-aeff-4118-bd3d-d070c1c83a88"
+					(reference "R11")
+					(unit 1)
+				)

Commit message: Final changes before manufacture.
Parts:
- C11, C12: footprint Capacitor_SMD:C_0805_2012Metric -> Capacitor_SMD:C_0603_1608Metric
Other:
- note added: "C3757764"
- note added: "C579454"
- note added: "MCP73831T-2ACI/OT C424093"
- note added: "Switches: JLC C513492 Manu: 2-1825910-7"
Changed lines of the file:
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@@
 		)
 	)
+	(text "Switches: JLC C513492 Manu: 2-1825910-7"
+		(exclude_from_sim no)
+		(at 137.414 172.974 0)
+		(effects
+			(font
+				(size 1.27 1.27)
+			)
+		)
+	)
+	(text "C3757764"
+		(exclude_from_sim no)
+		(at 38.862 109.474 0)
+		(effects
+			(font
+				(size 1.27 1.27)
+			)
+		)
+	)
 	(text "C5276598"
 		(exclude_from_sim no)
@@
 		)
 	)
+	(text "C579454"
+		(exclude_from_sim no)
+		(at 260.35 122.428 0)
+		(effects
+			(font
+				(size 1.27 1.27)
+			)
+		)
+	)
+	(text "MCP73831T-2ACI/OT\nC424093"
+		(exclude_from_sim no)
+		(at 39.37 167.132 0)
+		(effects
+			(font
+				(size 1.27 1.27)
+			)
+		)
+	)
 	(text "INT Push-Pull"
 		(exclude_from_sim no)
@@
 		(fields_autoplaced yes)
 		(property "Reference" "C11"
-			(at 275.59 93.345 0)
+			(at 275.59 92.7099 0)
 			(effects
 				(font
@@
 		)
 		(property "Value" "0.1uF"
-			(at 275.59 95.885 0)
+			(at 275.59 95.2499 0)
 			(effects
 				(font
@@
 			)
 		)
-		(property "Footprint" "Capacitor_SMD:C_0805_2012Metric"
+		(property "Footprint" "Capacitor_SMD:C_0603_1608Metric"
 			(at 272.7452 97.79 0)
 			(effects
@@
 		(fields_autoplaced yes)
 		(property "Reference" "C12"
-			(at 275.59 135.255 0)
+			(at 275.59 134.6199 0)
 			(effects
 				(font
@@
 		)
 		(property "Value" "0.1uF"
-			(at 275.59 137.795 0)
+			(at 275.59 137.1599 0)
 			(effects
 				(font
@@
 			)
 		)
-		(property "Footprint" "Capacitor_SMD:C_0805_2012Metric"
+		(property "Footprint" "Capacitor_SMD:C_0603_1608Metric"
 			(at 272.7452 139.7 0)
 			(effects
@@
 			)
 		)
-		(property "Description" "C306879"
+		(property "Description" ""
 			(at 34.29 53.34 0)
 			(effects
